File: pcb/alarmbuddy.sch (KiCad schematic (older format))
At the start: 20 parts, among them J1 10VAC, J4 3V3, J5 SENS1-3, J6 SENS4-6, J7 SENS7-9, J8 SENS10-12, J9 FTDI, U1 VXO7803-500, U3 ESP32-WROOM-32D

Commit message: v3
Connections:
- net +3V3: now also J9.3 (Pin_3); no longer J9.4 (Pin_4)
- net RTS: now also J9.1 (Pin_1); no longer J9.5 (Pin_5)
- net RX: now also J9.5 (Pin_5); no longer J9.2 (Pin_2)
- net TX: now also J9.4 (Pin_4); no longer J9.3 (Pin_3)
- net ~DTR: now also J9.2 (Pin_2); no longer J9.1 (Pin_1)
Other:
- moved on the sheet: J9
Changed lines of the file:
@@
 Wire Wire Line
 	1200 1250 1200 1325
-Text Label 1025 6150 0    39   ~ 0
+Text Label 1150 5750 0    39   ~ 0
 RTS
-Text Label 1025 6050 0    39   ~ 0
+Text Label 1150 5950 0    39   ~ 0
 3V3
-Text Label 1025 5950 0    39   ~ 0
+Text Label 1150 6050 0    39   ~ 0
 TX
-Text Label 1025 5850 0    39   ~ 0
+Text Label 1150 6150 0    39   ~ 0
 RX
-Text Label 1025 5750 0    39   ~ 0
+Text Label 1150 5850 0    39   ~ 0
 ~DTR
 $Comp
 L Connector_Generic:Conn_01x06 J9
 U 1 1 5E2F9BC4
-P 1425 5950
-F 0 "J9" H 1505 5942 50  0000 L CNN
-F 1 "FTDI" H 1505 5851 50  0000 L CNN
-F 2 "Connector_PinHeader_2.54mm:PinHeader_1x06_P2.54mm_Vertical" H 1425 5950 50  0001 C CNN
-F 3 "~" H 1425 5950 50  0001 C CNN
-	1    1425 5950
-	1    0    0    -1
-$EndComp
-Wire Wire Line
-	1225 6150 1025 6150
-Wire Wire Line
-	1225 6050 1025 6050
-Wire Wire Line
-	1225 5950 1025 5950
-Wire Wire Line
-	1225 5850 1025 5850
-Wire Wire Line
-	1225 5750 1025 5750
+P 1550 5950
+F 0 "J9" H 1630 5942 50  0000 L CNN
+F 1 "FTDI" H 1630 5851 50  0000 L CNN
+F 2 "Connector_PinHeader_2.54mm:PinHeader_1x06_P2.54mm_Vertical" H 1550 5950 50  0001 C CNN
+F 3 "~" H 1550 5950 50  0001 C CNN
+	1    1550 5950
+	1    0    0    -1
+$EndComp
 Wire Wire Line
 	5850 3100 6300 3100
@@
 Wire Wire Line
 	800  7600 750  7600
-$Comp
-L power:GND #PWR02
-U 1 1 5E3E817A
-P 1300 7450
-F 0 "#PWR02" H 1300 7200 50  0001 C CNN
-F 1 "GND" H 1305 7277 50  0000 C CNN
-F 2 "" H 1300 7450 50  0001 C CNN
-F 3 "" H 1300 7450 50  0001 C CNN
-	1    1300 7450
-	1    0    0    -1
-$EndComp
 Wire Wire Line
 	5950 3200 5850 3200
@@
 L power:GND #PWR?
 U 1 1 5E2A6A77
-P 1225 6250
+P 1200 6250
 AR Path="/5C5CDDE8/5E2A6A77" Ref="#PWR?"  Part="1"
 AR Path="/5E2A6A77" Ref="#PWR017"  Part="1"
 AR Path="/5E244F48/5E2A6A77" Ref="#PWR?"  Part="1"
-F 0 "#PWR017" H 1225 6000 50  0001 C CNN
-F 1 "GND" H 1230 6077 50  0000 C CNN
-F 2 "" H 1225 6250 50  0001 C CNN
-F 3 "" H 1225 6250 50  0001 C CNN
-	1    1225 6250
+F 0 "#PWR017" H 1200 6000 50  0001 C CNN
+F 1 "GND" H 1205 6077 50  0000 C CNN
+F 2 "" H 1200 6250 50  0001 C CNN
+F 3 "" H 1200 6250 50  0001 C CNN
+	1    1200 6250
 	1    0    0    -1
 $EndComp
@@
 Wire Wire Line
 	4350 1250 4700 1250
+Wire Wire Line
+	1350 5750 1150 5750
+Wire Wire Line
+	1350 5850 1150 5850
+Wire Wire Line
+	1350 5950 1150 5950
+Wire Wire Line
+	1350 6050 1150 6050
+Wire Wire Line
+	1350 6150 1150 6150
+Wire Wire Line
+	1350 6250 1200 6250
 $EndSCHEMATC

Commit message: docs
Other:
- note added: "GPIO2 needs to be \nlow or floating when \nbooting to flash \nproperly. Avoid using\nif possible."
Changed lines of the file:
@@
 Wire Wire Line
 	1350 6250 1200 6250
+Text Notes 4750 4000 0    50   ~ 0
+GPIO2 needs to be \nlow or floating when \nbooting to flash \nproperly. Avoid using\nif possible.
 $EndSCHEMATC

Commit message: esp32-s2 change
Parts:
- removed C7: 0.1uF, Capacitor_SMD:C_1206_3216Metric, symbol Device:C_Small
- removed J4: 3V3, TerminalBlock_Phoenix:TerminalBlock_Phoenix_PT-1,5-3-5.0-H_1x03_P5.00mm_Horizontal, symbol Connector:Screw_Terminal_01x03
- removed TP2: TP3V3, TestPoint:TestPoint_Pad_D2.0mm, symbol Connector:TestPoint
- removed U3: ESP32-WROOM-32D, RF_Module:ESP32-WROOM-32, symbol RF_Module:ESP32-WROOM-32D
- added C5: 10uF 50V, Capacitor_SMD:C_1206_3216Metric, symbol Device:C_Small
- added C6: 22uF 10V, Capacitor_SMD:C_1206_3216Metric, symbol Device:C_Small
- added J2: 12V, TerminalBlock_Phoenix:TerminalBlock_Phoenix_PT-1,5-2-5.0-H_1x02_P5.00mm_Horizontal, symbol Connector:Screw_Terminal_01x02
- added J4: 3V3, TerminalBlock_Phoenix:TerminalBlock_Phoenix_PT-1,5-2-5.0-H_1x02_P5.00mm_Horizontal, symbol Connector:Screw_Terminal_01x02
- added R1: 10K, Resistor_SMD:R_1206_3216Metric, symbol Device:R_Small
- added U2: ESP32-S2-WROVER, RF_Module:ESP32-S2-WROVER, symbol RF_Module:ESP32-S2-WROVER
- added U3: VXO-78XX, !Greg:VXO78-500, symbol !Custom:VXO78xx
Connections:
- net +3V3: now also R1.2, U2.2 (3V3)
- net 3V3_COMMON: now also J4.1 (Pin_1), J4.2 (Pin_2)
- net GND: now also C5.2, C6.2, U2.1 (GND), U2.26 (GND), U2.42 (GND), U2.43 (GND), U3.2 (GND)
- net RTS: now also U2.41 (EN)
- net RX: now also U2.37 (TXD0)
- net SENSOR1: now also U2.4 (IO01)
- net SENSOR10: now also U2.15 (IO12)
- net SENSOR11: now also U2.14 (IO11)
- net SENSOR12: now also U2.13 (IO10)
- net SENSOR2: now also U2.5 (IO02)
- net SENSOR3: now also U2.6 (IO03)
- net SENSOR4: now also U2.7 (IO04)
- net SENSOR5: now also U2.8 (IO05)
- net SENSOR6: now also U2.9 (IO06)
- net SENSOR7: now also U2.10 (IO07)
- net SENSOR8: now also U2.11 (IO08)
- net SENSOR9: now also U2.12 (IO09)
- net TX: now also U2.38 (RXD0)
- net ~DTR: now also U2.3 (IO00)
- net at C1.1, C2.1, C3.1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: now also C5.1, U3.1 (IN)
- new net: R1.1, U2.21 (IO18)
- new net +12V: C6.1, J2.1 (Pin_1), J2.2 (Pin_2), U3.3 (OUT)
- no-connect marks 17 -> 2
Other:
- note added: "GPIO11-18 = ADC2\nMust disable WiFi for ADC2"
- note added: "GPIO18 works as U1RXD and is in\n an uncertain state when the chip is powered on, \nwhich may affect the chip’s\nentry into download boot mode. \nTo solve this issue, add an \nexternal pull-up resistor."
- note added: "IO46/IO45 strapping pins\navoid or use with caution"
- note removed: "(already has small \n bypass caps)"
- note removed: "34/35 are\ninput only"
- note removed: "GPIO2 needs to be \nlow or floating when \nbooting to flash \nproperly. Avoid using\nif possible."
- moved on the sheet: C9, R5
